Commit message: ros2_control_edit_before_slam

File: wael_package/src/description/gazebo.xacro (robot description, xacro)
@@ -32,4 +32,7 @@
     <material>Gazebo/Yellow</material>
   </gazebo>
+  <gazebo reference="lidar_link">
+    <material>Gazebo/Black</material>
+  </gazebo>
 <!--WORKING DIFF DRIVE NO FRICTION FOR WHEELS REAR-->
 <gazebo>
@@ -48,16 +51,3 @@
     </plugin>
   </gazebo>
-  <!--MAke the rear wheels with no friction to let the robot move smoothley-->
-  <gazebo reference="rearwhl_l_link">
-    <mu1>0.0</mu1>
-    <mu2>0.0</mu2>
-    <kp>1e9</kp>
-    <kd>1</kd>
-  </gazebo>
-  <gazebo reference="rearwhl_r_link">
-    <mu1>0.0</mu1>
-    <mu2>0.0</mu2>
-    <kp>1e9</kp>
-    <kd>1</kd>
-  </gazebo>
 </robot>

File: wael_package/src/description/sensors.xacro (robot description, xacro)
@@ -75,29 +75,4 @@
     <origin xyz="0 0 0.01"/>
   </joint>
-  <!--Lidar Sensor-->
-  <link name="lidar_link">
-  <inertial>
-    <origin xyz="0 0 0" rpy="0 0 0"/>
-    <mass value="0.125"/>
-    <inertia ixx="0.001"  ixy="0"  ixz="0" iyy="0.001" iyz="0" izz="0.001" />
-  </inertial>
-  <collision>
-    <origin xyz="0 0 0" rpy="0 0 0"/>
-    <geometry>
-       <cylinder radius="0.0508" length="0.055"/>
-    </geometry>
-  </collision>
-  <visual>
-    <origin xyz="0 0 0" rpy="0 0 0"/>
-    <geometry>
-       <cylinder radius="0.0508" length="0.055"/>
-    </geometry>
-  </visual>
-  </link>
-  <joint name="lidar_joint" type="fixed">
-    <parent link="top_layer_link"/>
-    <child link="lidar_link"/>
-    <origin xyz="0 0 0.12" rpy="0 0 0"/>
-  </joint>
   <!--IMU Gazebo-->
   <gazebo reference="imu_link">
@@ -169,38 +144,3 @@
    </sensor>
   </gazebo>
-  <!--Lidar Gazibo-->
-  <gazebo reference="lidar_link">
-   <sensor name="lidar" type="ray">
-    <always_on>true</always_on>
-    <visualize>true</visualize>
-    <update_rate>5</update_rate>
-    <ray>
-      <scan>
-        <horizontal>
-          <samples>360</samples>
-          <resolution>1.000000</resolution>
-          <min_angle>0.000000</min_angle>
-          <max_angle>6.280000</max_angle>
-        </horizontal>
-      </scan>
-      <range>
-        <min>0.120000</min>
-        <max>3.5</max>
-        <resolution>0.015000</resolution>
-      </range>
-      <noise>
-        <type>gaussian</type>
-        <mean>0.0</mean>
-        <stddev>0.01</stddev>
-      </noise>
-    </ray>
-    <plugin name="scan" filename="libgazebo_ros_ray_sensor.so">
-      <ros>
-        <remapping>~/out:=scan</remapping>
-      </ros>
-      <output_type>sensor_msgs/LaserScan</output_type>
-      <frame_name>lidar_link</frame_name>
-    </plugin>
-   </sensor>
-  </gazebo>
 </robot>

File: wael_package/src/description/wheels.xacro (robot description, xacro)
@@ -38,3 +38,16 @@
   <xacro:wheel fixedOrCont="fixed" prefix="rearwhl_l" x_reflect="-1" y_reflect="1" />
   <xacro:wheel fixedOrCont="fixed" prefix="rearwhl_r" x_reflect="-1" y_reflect="-1" />
+  <!--MAke the rear wheels with no friction to let the robot move smoothley-->
+  <gazebo reference="rearwhl_l_link">
+    <mu1>0.0</mu1>
+    <mu2>0.0</mu2>
+    <kp>1e9</kp>
+    <kd>1</kd>
+  </gazebo>
+  <gazebo reference="rearwhl_r_link">
+    <mu1>0.0</mu1>
+    <mu2>0.0</mu2>
+    <kp>1e9</kp>
+    <kd>1</kd>
+  </gazebo>
 </robot>

Commit message: 4th commit, SLAM Working with both gazebo and ros2_control plugins

File: wael_package/src/description/gazebo.xacro (robot description, xacro)
@@ -32,7 +32,10 @@
     <material>Gazebo/Yellow</material>
   </gazebo>
-  <gazebo reference="lidar_link">
+  <gazebo reference="imu_link">
     <material>Gazebo/Black</material>
   </gazebo>
+  <!-- <gazebo reference="lidar_link">
+    <material>Gazebo/Black</material>
+  </gazebo> -->
 <!--WORKING DIFF DRIVE NO FRICTION FOR WHEELS REAR-->
 <gazebo>
@@ -51,3 +54,91 @@
     </plugin>
   </gazebo>
+    <!--IMU sensor-->
+  <link name="imu_link">
+  <visual>
+    <geometry>
+      <box size="0.01 0.005 0.0001"/>
+    </geometry>
+  </visual>
+  <collision>
+    <geometry>
+      <box size="0.01 0.01 0.01"/>
+    </geometry>
+  </collision>
+  <xacro:box_inertia m="0.001" w="0.01" d="0.005" h="0.0001"/>
+  </link>
+  <joint name="imu_joint" type="fixed">
+    <parent link="base_link"/>
+    <child link="imu_link"/>
+    <origin xyz="0 0 0.02"/>
+  </joint>
+  <!--IMU Gazebo-->
+  <gazebo reference="imu_link">
+   <sensor name="imu_sensor" type="imu">
+    <plugin filename="libgazebo_ros_imu_sensor.so" name="imu_plugin">
+      <ros>
+        <namespace>/demo</namespace>
+        <remapping>~/out:=imu</remapping>
+      </ros>
+      <initial_orientation_as_reference>false</initial_orientation_as_reference>
+    </plugin>
+    <always_on>true</always_on>
+    <update_rate>100</update_rate>
+    <visualize>true</visualize>
+    <imu>
+      <angular_velocity>
+        <x>
+          <noise type="gaussian">
+            <mean>0.0</mean>
+            <stddev>2e-4</stddev>
+            <bias_mean>0.0000075</bias_mean>
+            <bias_stddev>0.0000008</bias_stddev>
+          </noise>
+        </x>
+        <y>
+          <noise type="gaussian">
+            <mean>0.0</mean>
+            <stddev>2e-4</stddev>
+            <bias_mean>0.0000075</bias_mean>
+            <bias_stddev>0.0000008</bias_stddev>
+          </noise>
+        </y>
+        <z>
+          <noise type="gaussian">
+            <mean>0.0</mean>
+            <stddev>2e-4</stddev>
+            <bias_mean>0.0000075</bias_mean>
+            <bias_stddev>0.0000008</bias_stddev>
+          </noise>
+        </z>
+      </angular_velocity>
+      <linear_acceleration>
+        <x>
+          <noise type="gaussian">
+            <mean>0.0</mean>
+            <stddev>1.7e-2</stddev>
+            <bias_mean>0.1</bias_mean>
+            <bias_stddev>0.001</bias_stddev>
+          </noise>
+        </x>
+        <y>
+          <noise type="gaussian">
+            <mean>0.0</mean>
+            <stddev>1.7e-2</stddev>
+            <bias_mean>0.1</bias_mean>
+            <bias_stddev>0.001</bias_stddev>
+          </noise>
+        </y>
+        <z>
+          <noise type="gaussian">
+            <mean>0.0</mean>
+            <stddev>1.7e-2</stddev>
+            <bias_mean>0.1</bias_mean>
+            <bias_stddev>0.001</bias_stddev>
+          </noise>
+        </z>
+      </linear_acceleration>
+    </imu>
+   </sensor>
+  </gazebo>
 </robot>

File: wael_package/src/description/sensors.xacro (robot description, xacro)
@@ -29,31 +29,4 @@
     </gazebo>
 </robot>
-  <!-- Diff Drive Plugin -->
-  <gazebo>
-    <plugin name="diff_drive" filename="libgazebo_ros_diff_drive.so">
-      <ros>
-        <namespace>/</namespace>
-      </ros>
-      <!-- wheels -->
-      <left_joint>drivewhl_l_joint</left_joint>
-      <right_joint>drivewhl_r_joint</right_joint>
-      <left2_joint>rearwhl_l_joint</left2_joint>
-      <right2_joint>rearwhl_r_joint</right2_joint>
-      <!-- kinematics -->
-      <wheel_separation>0.2</wheel_separation>
-      <wheel_diameter>0.12</wheel_diameter>
-      <!--Try to change it-->
-      <!-- limits -->
-      <max_wheel_torque>20</max_wheel_torque>
-      <max_wheel_acceleration>1.0</max_wheel_acceleration>
-      <!-- output -->
-      <publish_odom>true</publish_odom>
-      <publish_odom_tf>true</publish_odom_tf>
-      <publish_wheel_tf>true</publish_wheel_tf>
-      <odometry_frame>odom</odometry_frame>
-      <robot_base_frame>base_link</robot_base_frame>
-      <!--Try to change it-->
-    </plugin>
-  </gazebo>
   <!--IMU sensor-->
   <link name="imu_link">

File: wael_package/src/description/wheels.xacro (robot description, xacro)
@@ -7,4 +7,7 @@
   <xacro:property name="wheel_zoff" value="0.0"/>
   <xacro:property name="wheel_xoff" value="0.0"/>
+<!-- keep in mind if there is problem in slippery between Gazebo and RVIZ
+  you can change the collision gemetry of the wheels into sphere without toaching the visuals
+  Last time I checked the rotation it is pretty good no need -->
   <!-- Wheels Xacro and instances-->
   <xacro:macro name="wheel" params="prefix x_reflect y_reflect fixedOrCont">

Commit message: fifth commit: NAV2 running with amcl (loaded map)

File: wael_package/src/description/gazebo.xacro (robot description, xacro)
@@ -54,91 +54,3 @@
     </plugin>
   </gazebo>
-    <!--IMU sensor-->
-  <link name="imu_link">
-  <visual>
-    <geometry>
-      <box size="0.01 0.005 0.0001"/>
-    </geometry>
-  </visual>
-  <collision>
-    <geometry>
-      <box size="0.01 0.01 0.01"/>
-    </geometry>
-  </collision>
-  <xacro:box_inertia m="0.001" w="0.01" d="0.005" h="0.0001"/>
-  </link>
-  <joint name="imu_joint" type="fixed">
-    <parent link="base_link"/>
-    <child link="imu_link"/>
-    <origin xyz="0 0 0.02"/>
-  </joint>
-  <!--IMU Gazebo-->
-  <gazebo reference="imu_link">
-   <sensor name="imu_sensor" type="imu">
-    <plugin filename="libgazebo_ros_imu_sensor.so" name="imu_plugin">
-      <ros>
-        <namespace>/demo</namespace>
-        <remapping>~/out:=imu</remapping>
-      </ros>
-      <initial_orientation_as_reference>false</initial_orientation_as_reference>
-    </plugin>
-    <always_on>true</always_on>
-    <update_rate>100</update_rate>
-    <visualize>true</visualize>
-    <imu>
-      <angular_velocity>
-        <x>
-          <noise type="gaussian">
-            <mean>0.0</mean>
-            <stddev>2e-4</stddev>
-            <bias_mean>0.0000075</bias_mean>
-            <bias_stddev>0.0000008</bias_stddev>
-          </noise>
-        </x>
-        <y>
-          <noise type="gaussian">
-            <mean>0.0</mean>
-            <stddev>2e-4</stddev>
-            <bias_mean>0.0000075</bias_mean>
-            <bias_stddev>0.0000008</bias_stddev>
-          </noise>
-        </y>
-        <z>
-          <noise type="gaussian">
-            <mean>0.0</mean>
-            <stddev>2e-4</stddev>
-            <bias_mean>0.0000075</bias_mean>
-            <bias_stddev>0.0000008</bias_stddev>
-          </noise>
-        </z>
-      </angular_velocity>
-      <linear_acceleration>
-        <x>
-          <noise type="gaussian">
-            <mean>0.0</mean>
-            <stddev>1.7e-2</stddev>
-            <bias_mean>0.1</bias_mean>
-            <bias_stddev>0.001</bias_stddev>
-          </noise>
-        </x>
-        <y>
-          <noise type="gaussian">
-            <mean>0.0</mean>
-            <stddev>1.7e-2</stddev>
-            <bias_mean>0.1</bias_mean>
-            <bias_stddev>0.001</bias_stddev>
-          </noise>
-        </y>
-        <z>
-          <noise type="gaussian">
-            <mean>0.0</mean>
-            <stddev>1.7e-2</stddev>
-            <bias_mean>0.1</bias_mean>
-            <bias_stddev>0.001</bias_stddev>
-          </noise>
-        </z>
-      </linear_acceleration>
-    </imu>
-   </sensor>
-  </gazebo>
 </robot>
